Commit message: Changes to pose est, car data and URDF, configs
Changed the pose estimation and car data publisher to use the
ROS time via rate.sleep(), was previously using steady_clock in
c++ chrono lib. Updated URDF because we used the REAR left radar
due to cable length issues.  Also updated some config files
from Rviz and for tuning (YAMLs).

File: urdf/car_gps_test.urdf (robot description, URDF)
Before this commit: robot car, 14 links, 13 joints
Joints:
- joint front_left_radar_joint: origin xyz=2.2 0.7 0.4 rpy=0 0 ${(pi/180)*40} -> xyz=2.2 0.7 0.4 rpy=0 0 ${(pi/180)*90}
- joint front_left_wheel_joint: axis 1 0 0 -> 0 1 0
- joint front_right_wheel_joint: axis 1 0 0 -> 0 1 0
- joint rear_left_radar_joint: origin xyz=-2.5 0.7 0.4 rpy=0 0 ${(pi/180)*(180-40)} -> xyz=-2.5 0.7 0.4 rpy=0 0 ${(pi/180)*(90)}
- joint rear_left_wheel_joint: axis 1 0 0 -> 0 1 0
- joint rear_right_wheel_joint: axis 1 0 0 -> 0 1 0

Commit message: Post auto show demo dump of changes

File: urdf/car_gps_test.urdf (robot description, URDF)
Before this commit: robot car, 14 links, 13 joints
Joints:
- joint front_left_radar_joint: origin xyz=2.2 0.7 0.4 rpy=0 0 ${(pi/180)*40} -> xyz=2.2 0.7 0.4 rpy=0 0 ${(pi/180)*90}
- joint rear_left_radar_joint: origin xyz=-2.5 0.7 0.4 rpy=0 0 ${(pi/180)*(180-40)} -> xyz=-2.5 0.7 0.4 rpy=0 0 ${(pi/180)*(90)}
