Commit message: Minor change to bobcat URDF, add new separate launch file

File: urdf/bobcat.urdf (robot description, URDF)
Before this commit: robot bobcat, 4 links, 3 joints
Links:
- removed link left_radar_link
- removed link right_radar_link
- added link front_right_radar_link, mass 1; visual mesh filename=package://radar_slam/meshes/kanza79.stl scale=1.0 1.0 1.0
- added link rear_left_radar_link, mass 1; visual mesh filename=package://radar_slam/meshes/kanza79.stl scale=1.0 1.0 1.0
Joints:
- removed joint left_radar_joint
- removed joint right_radar_joint
- added joint front_right_radar_joint: type fixed, parent chassis, child front_right_radar_link, origin xyz=-0.55 0.2 1.0 rpy=0 0 ${1.0*pi}
- added joint rear_left_radar_joint: type fixed, parent chassis, child rear_left_radar_link, origin xyz=0.55 0.2 1.0 rpy=0 0 ${0.0*pi}

Commit message: Minor change to bobcat URDF
Fixed bobcat URDF to have x axis forward as per ROS convention
(see http://www.ros.org/reps/rep-0103.html).

File: urdf/bobcat.urdf (robot description, URDF)
Before this commit: robot bobcat, 4 links, 3 joints
Joints:
- joint front_right_radar_joint: origin xyz=-0.55 0.2 1.0 rpy=0 0 ${1.0*pi} -> xyz=0.2 -0.55 1.0 rpy=0 0 ${-0.5*pi}
- joint rear_left_radar_joint: origin xyz=0.55 0.2 1.0 rpy=0 0 ${0.0*pi} -> xyz=0.2 0.55 1.0 rpy=0 0 ${0.5*pi}
